File: kicad/cercane/cercane.kicad_pcb (KiCad board)
At the start: 2 copper layers, 34.3 x 27.9 mm, 4 parts, among them J1 Conn_02x03_Odd_Even, U1 ATtiny45-20PU, U2 NRF24L01_Breakout

Commit message: combed tracks
Routing:
- net /RST: track 44.1 -> 50.4 mm
- net /MISO: track 32.0 -> 37.1 mm
- net /MOSI: track 21.9 -> 25.9 mm
